Commit message: Add real physical data, and modify for it

File: balancingkit_description/urdf/balancingkit.urdf (robot description, URDF)
Before this commit: robot balancingkit, 3 links, 2 joints
Links:
- added link battery_cover, mass 0.0135409963305; collision mesh filename=package://balancingkit_description/meshes/stl/body/balboa_b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; visual mesh filename=package://balancingkit_description/meshes/stl/body/balboa_b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
- added link circuit_board, mass 0.0116038891251; collision mesh filename=package://balancingkit_description/meshes/stl/body/balboa_b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; visual mesh filename=package://balancingkit_description/meshes/stl/body/balboa_b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
- link base_link: mass None -> 0.0687016219743; geometry collision mesh filename=package://balancingkit_description/meshes/stl/body/balboa_b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; visual mesh filename=package://balancingkit_description/meshes/stl/body/balboa_b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
- link left-wheel: mass None -> 0.0192200809141; geometry collision mesh filename=package://balancingkit_description/meshes/stl/wheel/balboa_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; visual mesh filename=package://balancingkit_description/meshes/stl/wheel/balboa_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
- link right-wheel: mass None -> 0.0192200809141; geometry collision mesh filename=package://balancingkit_description/meshes/stl/wheel/balboa_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; visual mesh filename=package://balancingkit_description/meshes/stl/wheel/balboa_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
Joints:
- added joint battery_cover_joint: type fixed, parent base_link, child battery_cover, origin xyz=0 0 0 rpy=0 0 0, axis 0 0 0
- added joint circuit_board_joint: type fixed, parent base_link, child circuit_board, origin xyz=0 0 0 rpy=0 0 0, axis 0 0 0
- joint left-wheel_joint: origin xyz=-0.051 0 0 rpy=0 0 0 -> xyz=0 -0.02 -0.0097 rpy=0 0 0
- joint right-wheel_joint: origin xyz=0.051 0 0 rpy=0 0 0 -> xyz=0 -0.02 -0.0097 rpy=0 0 0

Commit message: Modify link origin

File: balancingkit_description/urdf/balancingkit.urdf (robot description, URDF)
Before this commit: robot balancingkit, 5 links, 4 joints
Links:
- removed link left-wheel
- removed link right-wheel
- added link base_footprint
- added link left_wheel, mass 0.0192200809141; collision mesh filename=package://balancingkit_description/meshes/stl/wheel/balboa_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; visual mesh filename=package://balancingkit_description/meshes/stl/wheel/balboa_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
- added link right_wheel, mass 0.0192200809141; collision mesh filename=package://balancingkit_description/meshes/stl/wheel/balboa_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; visual mesh filename=package://balancingkit_description/meshes/stl/wheel/balboa_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
Joints:
- removed joint left-wheel_joint
- removed joint right-wheel_joint
- added joint foot_print_joint: type fixed, parent base_footprint, child base_link, origin xyz=0 0.02 0.0097 rpy=0 0 0
- added joint left_wheel_joint: type continuous, parent base_link, child left_wheel, origin xyz=-0.051 -0.02 -0.0097 rpy=0 0 0, axis 1 0 0
- added joint right_wheel_joint: type continuous, parent base_link, child right_wheel, origin xyz=0.051 -0.02 -0.0097 rpy=0 0 0, axis 1 0 0
