Commit message: Modify

File: balancingkit_description/urdf/balancingkit.urdf.xacro (robot description, xacro)
@@ -1,19 +1,22 @@
 <?xml version="1.0"?>
-<robot name="balancingkit_on_gazebo" xmlns:xacro="http://ros.org/wiki/xacro">
+<robot name="balancingkit_on_gazebo"
+       xmlns:controller="http://playerstage.sourceforge.net/gazebo/xmlschema/#controller"
+       xmlns:interface="http://playerstage.sourceforge.net/gazebo/xmlschema/#interface"
+       xmlns:xacro="http://ros.org/wiki/xacro">
   <xacro:include filename="$(find balancingkit_description)/urdf/body/body.urdf.xacro"/>
   <xacro:include filename="$(find balancingkit_description)/urdf/wheel/wheel.urdf.xacro"/>
   <!-- =============== Link & Joint =============== -->
   <!-- Base -->
-  <link name="base_link"/>
-  <xacro:base parent="base_link">
-    <origin xyz="0 0 0.040"/>
+  <link name="base_footprint"/>
+  <xacro:base parent="base_footprint">
+    <origin xyz="0 0.02 0.0097"/>
   </xacro:base>
   <!-- Wheel -->
   <xacro:wheel prefix="right" parent="base_link">
-    <origin xyz="0.051 0 0" rpy="0 0 0"/>
+    <origin xyz="0.051 -0.02 -0.0097" rpy="0 0 0"/>
     <axis xyz="1 0 0"/>
   </xacro:wheel>
   <xacro:wheel prefix="left" parent="base_link">
-    <origin xyz="-0.051 0 0" rpy="0 0 0"/>
+    <origin xyz="-0.051 -0.02 -0.0097" rpy="0 0 0"/>
     <axis xyz="1 0 0"/>
   </xacro:wheel>

File: balancingkit_description/urdf/body/body.urdf.xacro (robot description, xacro)
@@ -1,5 +1,5 @@
 <?xml version="1.0"?>
 <robot xmlns:xacro="http://ros.org/wiki/xacro">
-  <xacro:include filename="$(find raspimouse_description)/urdf/body/body.gazebo.xacro"/>
+  <xacro:include filename="$(find balancingkit_description)/urdf/body/body.gazebo.xacro"/>
   <xacro:property name="M_PI" value="3.1415926535897931" />
   <xacro:property name="velocity_scale_factor" value="1.0"/>
@@ -13,10 +13,10 @@
       <visual>
         <geometry>
-          <mesh filename="package://raspimouse_description/meshes/dae/body/RasPiMouse_body.dae"/>
+          <mesh filename="package://balancingkit_description/meshes/stl/body/balboa_balancing_robot_kit_body_chassis_m.stl"/>
         </geometry>
       </visual>
       <collision>
         <geometry>
-          <mesh filename="package://raspimouse_description/meshes/dae/body/RasPiMouse_body.dae"/>
+          <mesh filename="package://balancingkit_description/meshes/stl/body/balboa_balancing_robot_kit_body_chassis_m.stl"/>
         </geometry>
       </collision>
@@ -29,7 +29,7 @@
         <!-- <origin xyz="&#45;0.005075 &#45;0.000427 0.029879"/> -->
         <!-- virtual origin -->
-        <origin xyz="-0.001 0.0 0.029879"/>
-        <mass value="0.7186"/>
-        <inertia ixx="0.001238161833" ixy="0.000000904986" iyy="0.001368529369" ixz="0.000100297310" iyz="0.000022118177" izz="0.000784319117"/>
+        <!-- <origin xyz="-0.001 0.0 0.029879"/> -->
+        <mass value="0.0687016219743" />
+        <inertia ixx="0.00004951341871460000" ixy="0.00000045970330081100" ixz="0.00000003906431665210" iyy="0.00007420445567420000" iyz="0.00000188480164726000" izz="0.00011062967861500000" />
       </inertial>
     </link>

File: balancingkit_description/urdf/wheel/wheel.urdf.xacro (robot description, xacro)
@@ -1,10 +1,9 @@
 <?xml version="1.0"?>
 <robot xmlns:xacro="http://ros.org/wiki/xacro">
-  <xacro:include filename="$(find raspimouse_description)/urdf/wheel/wheel.transmission.xacro"/>
-  <xacro:include filename="$(find raspimouse_description)/urdf/wheel/wheel.gazebo.xacro"/>
-  <!-- <property name="wheel_radius" value="0.0239"/> -->
-  <property name="wheel_radius" value="0.0249"/>
-  <property name="wheel_length" value="0.01"/>
-  <property name="wheel_mass" value="0.0113"/>
+  <xacro:include filename="$(find balancingkit_description)/urdf/wheel/wheel.transmission.xacro"/>
+  <xacro:include filename="$(find balancingkit_description)/urdf/wheel/wheel.gazebo.xacro"/>
+  <property name="wheel_radius" value="0.03825"/>
+  <property name="wheel_length" value="0.01"/> <!-- width? -->
+  <property name="wheel_mass" value="0.0192200809141"/>
   <xacro:macro name="wheel" params="prefix parent *joint_origin *joint_axis">
   <joint name="${prefix}_wheel_joint" type="continuous">
@@ -13,5 +12,5 @@
     <parent link="${parent}"/>
     <child link="${prefix}_wheel"/>
-    <limit effort="70" velocity="15"/>
+    <limit effort="70" velocity="15"/> <!-- TODO Need to calculate -->
     <safety_controller  k_velocity="10" />
     <dynamics damping="1.0" friction="1.0" />

Commit message: Modify xacro files

File: balancingkit_description/urdf/balancingkit.urdf.xacro (robot description, xacro)
@@ -27,15 +27,15 @@
   <!-- VelocityJointInterface: requires position, velocity -->
   <!-- for DiffDriveController -->
-<!--   <xacro:wheel_trans prefix="right" interface="VelocityJointInterface"/> -->
-<!--   <xacro:wheel_trans prefix="left" interface="VelocityJointInterface"/> -->
+  <xacro:wheel_trans prefix="right" interface="VelocityJointInterface"/>
+  <xacro:wheel_trans prefix="left" interface="VelocityJointInterface"/>
   <!-- EffortJointInterface: requires position, velocity, effort -->
   <!-- <xacro:wheel_trans prefix="right" interface="EffortJointInterface"/> -->
   <!-- <xacro:wheel_trans prefix="left" interface="EffortJointInterface"/>  -->
   <!-- =============== Gazebo =============== -->
-<!--     <gazebo> -->
-<!--       <plugin name="gazebo_ros_control" filename="libgazebo_ros_control.so"> -->
-<!--         <robotNamespace>balancingkit_on_gazebo</robotNamespace> -->
-<!--       </plugin> -->
-<!--     </gazebo> -->
+  <gazebo>
+    <plugin name="gazebo_ros_control" filename="libgazebo_ros_control.so">
+      <robotNamespace>balancingkit_on_gazebo</robotNamespace>
+    </plugin>
+  </gazebo>
   <!-- Base -->
   <xacro:base_gazebo/>

File: balancingkit_description/urdf/wheel/wheel.urdf.xacro (robot description, xacro)
@@ -19,5 +19,5 @@
     <visual>
       <geometry>
-        <mesh filename="package://raspimouse_description/meshes/dae/wheel/RasPiMouse_wheel.dae"/>
+        <mesh filename="package://balancingkit_description/meshes/stl/wheel/balboa_balancing_robot_kit_wheel_${prefix}_m.stl"/>
       </geometry>
     </visual>
@@ -25,12 +25,11 @@
       <!-- <insert_block name="joint_origin"/> -->
         <geometry>
-          <!-- <cylinder radius="${wheel_radius}" length="${wheel_length}"/> -->
-          <mesh filename="package://raspimouse_description/meshes/dae/wheel/RasPiMouse_wheel.dae"/>
+          <mesh filename="package://balancingkit_description/meshes/stl/wheel/balboa_balancing_robot_kit_wheel_${prefix}_m.stl"/>
         </geometry>
     </collision>
       <inertial>
-        <origin xyz="-0.000107 0 0.002875"/>
+        <origin xyz="0.051 0.02 0.0097" rpy="0 0 0"/><!-- TODO Need to confirm if both wheels have same origin -->
         <mass value="${wheel_mass}"/>
-        <inertia ixx="0.000002208187" ixy="0.000000000001" iyy="0.00000218412" ixz="0.000000004787" iyz="0.000000000003" izz="0.000004078299"/>
+        <inertia ixx="0.000021836231232000" ixy="0.000000000014016411" ixz="-0.000000000002704489" iyy="0.000011052671184900" iyz="-0.000000000002905832" izz="0.000011048923704800" />
       </inertial>
   </link>

Commit message: Modify

File: balancingkit_description/urdf/balancingkit.urdf.xacro (robot description, xacro)
@@ -1,46 +1 @@
-<?xml version="1.0"?>
-<robot name="balancingkit_on_gazebo"
-       xmlns:controller="http://playerstage.sourceforge.net/gazebo/xmlschema/#controller"
-       xmlns:interface="http://playerstage.sourceforge.net/gazebo/xmlschema/#interface"
-       xmlns:xacro="http://ros.org/wiki/xacro">
-  <xacro:include filename="$(find balancingkit_description)/urdf/body/body.urdf.xacro"/>
-  <xacro:include filename="$(find balancingkit_description)/urdf/wheel/wheel.urdf.xacro"/>
-  <!-- =============== Link & Joint =============== -->
-  <!-- Base -->
-  <link name="base_footprint"/>
-  <xacro:base parent="base_footprint">
-    <origin xyz="0 0.02 0.0097"/>
-  </xacro:base>
-  <!-- Wheel -->
-  <xacro:wheel prefix="right" parent="base_link">
-    <origin xyz="0.051 -0.02 -0.0097" rpy="0 0 0"/>
-    <axis xyz="1 0 0"/>
-  </xacro:wheel>
-  <xacro:wheel prefix="left" parent="base_link">
-    <origin xyz="-0.051 -0.02 -0.0097" rpy="0 0 0"/>
-    <axis xyz="1 0 0"/>
-  </xacro:wheel>
-  <!-- ===============  Transmission =============== -->
-  <!-- PositionJointInterface: requires position -->
-  <!-- <xacro:wheel_trans prefix="right" interface="PositionJointInterface"/> -->
-  <!-- <xacro:wheel_trans prefix="left" interface="PositionJointInterface"/>  -->
-  <!-- VelocityJointInterface: requires position, velocity -->
-  <!-- for DiffDriveController -->
-  <xacro:wheel_trans prefix="right" interface="VelocityJointInterface"/>
-  <xacro:wheel_trans prefix="left" interface="VelocityJointInterface"/>
-  <!-- EffortJointInterface: requires position, velocity, effort -->
-  <!-- <xacro:wheel_trans prefix="right" interface="EffortJointInterface"/> -->
-  <!-- <xacro:wheel_trans prefix="left" interface="EffortJointInterface"/>  -->
-  <!-- =============== Gazebo =============== -->
-  <gazebo>
-    <plugin name="gazebo_ros_control" filename="libgazebo_ros_control.so">
-      <robotNamespace>balancingkit_on_gazebo</robotNamespace>
-    </plugin>
-  </gazebo>
-  <!-- Base -->
-  <xacro:base_gazebo/>
-  <!-- Wheel -->
-  <xacro:wheel_gazebo prefix="right"/>
-  <xacro:wheel_gazebo prefix="left"/>
-  <balancingkit_on_gazebo/>
-</robot>
+../robots/balancingkit.urdf.xacro
