Commit message: Modify

File: balancingkit_description/urdf/body/body.urdf.xacro (robot description, xacro)
@@ -29,5 +29,5 @@
         <!-- <origin xyz="&#45;0.005075 &#45;0.000427 0.029879"/> -->
         <!-- virtual origin -->
-        <!-- <origin xyz="-0.001 0.0 0.029879"/> -->
+        <!-- TODO<origin xyz="-0.001 0.0 0.029879"/> -->
         <mass value="0.0687016219743" />
         <inertia ixx="0.00004951341871460000" ixy="0.00000045970330081100" ixz="0.00000003906431665210" iyy="0.00007420445567420000" iyz="0.00000188480164726000" izz="0.00011062967861500000" />

Commit message: Add cirquit boad and battery cover to body_xacro

File: balancingkit_description/urdf/body/body.urdf.xacro (robot description, xacro)
@@ -34,4 +34,48 @@
       </inertial>
     </link>
+    <joint name="circuit_board_joint" type="fixed">
+      <origin xyz="0 0 0" rpy="0 0 0"/>
+      <axis xyz="0 0 0"/>
+      <parent link="base_link"/>
+      <child link="circuit_board"/>
+    </joint>
+    <link name="circuit_board">
+      <inertial>
+        <mass value="0.0116038891251" />
+        <inertia ixx="0.00000000181524184545" ixy="-0.00000000011398958073" ixz="0.00000000001336676747" iyy="0.00000000181524184545" iyz="0.00000000001336676747" izz="0.00000000290410460112" />
+      </inertial>
+      <visual>
+        <geometry>
+          <mesh filename="package://balancingkit_description/meshes/stl/body/balboa_balancing_robot_kit_body_bal01a01_m.stl"/>
+        </geometry>
+      </visual>
+      <collision>
+        <geometry>
+          <mesh filename="package://balancingkit_description/meshes/stl/body/balboa_balancing_robot_kit_body_bal01a01_m.stl"/>
+        </geometry>
+      </collision>
+    </link>
+    <joint name="battery_cover_joint" type="fixed">
+      <origin xyz="0 0 0" rpy="0 0 0"/>
+      <axis xyz="0 0 0"/>
+      <parent link="base_link"/>
+      <child link="battery_cover"/>
+    </joint>
+    <link name="battery_cover">
+      <inertial>
+        <mass value="0.0135409963305" />
+        <inertia ixx="0.000009581429872300" ixy="-0.000000000605271997" ixz="0.000000000019527174" iyy="0.000003388820896330" iyz="-0.000000230335514201" izz="0.000012756434222000" />
+      </inertial>
+      <visual>
+        <geometry>
+          <mesh filename="package://balancingkit_description/meshes/stl/body/balboa_balancing_robot_kit_body_battery-cover_m.stl"/>
+        </geometry>
+      </visual>
+      <collision>
+        <geometry>
+          <mesh filename="package://balancingkit_description/meshes/stl/body/balboa_balancing_robot_kit_body_battery-cover_m.stl"/>
+        </geometry>
+      </collision>
+    </link>
   </xacro:macro>
 </robot>
