Commit message: Add color to stl

File: balancingkit_description/urdf/body/body.gazebo.xacro (robot description, xacro)
@@ -6,6 +6,17 @@
       <!-- <mu1 value="0.05" /> -->
       <!-- <mu2 value="0.05" /> -->
-      <mu1>0.05</mu1>
-      <mu2>0.05</mu2>
+      <material>Gazebo/DarkGrey</material>
+      <mu1>0.05</mu1> <!-- Coefficient of Friction -->
+      <mu2>0.05</mu2> <!-- Coefficient of Friction -->
+    </gazebo>
+    <gazebo reference="circuit_board">
+      <material>Gazebo/Green</material>
+      <mu1>0.05</mu1> <!-- Coefficient of Friction -->
+      <mu2>0.05</mu2> <!-- Coefficient of Friction -->
+    </gazebo>
+    <gazebo reference="battery_cover">
+      <material>Gazebo/DarkGrey</material>
+      <mu1>0.05</mu1> <!-- Coefficient of Friction -->
+      <mu2>0.05</mu2> <!-- Coefficient of Friction -->
     </gazebo>
   </xacro:macro>

File: balancingkit_description/urdf/wheel/wheel.gazebo.xacro (robot description, xacro)
@@ -6,4 +6,5 @@
       <!--   <mu1 value="0.8" /> -->
       <!--   <mu2 value="0.8" /> -->
+      <material>Gazebo/DarkGrey</material>
       <mu1>10.0</mu1>
       <mu2>10.0</mu2>
