Commit message: Fixed wheel origin

File: balancingkit_description/robots/balancingkit.urdf.xacro (robot description, xacro)
@@ -14,9 +14,9 @@
   <!-- Wheel -->
   <xacro:wheel prefix="right" parent="base_link">
-    <origin xyz="0.051 -0.02 -0.0097" rpy="0 0 0"/>
+    <origin xyz="0 0 0.0005" rpy="0 0 0"/>
     <axis xyz="1 0 0"/>
   </xacro:wheel>
   <xacro:wheel prefix="left" parent="base_link">
-    <origin xyz="-0.051 -0.02 -0.0097" rpy="0 0 0"/>
+    <origin xyz="0 0 0.0005" rpy="0 0 0"/>
     <axis xyz="1 0 0"/>
   </xacro:wheel>

File: balancingkit_description/urdf/wheel/wheel.urdf.xacro (robot description, xacro)
@@ -29,5 +29,4 @@
     </collision>
       <inertial>
-        <origin xyz="0.051 0.02 0.0097" rpy="0 0 0"/><!-- TODO Need to confirm if both wheels have same origin -->
         <mass value="${wheel_mass}"/>
         <inertia ixx="0.000021836231232000" ixy="0.000000000014016411" ixz="-0.000000000002704489" iyy="0.000011052671184900" iyz="-0.000000000002905832" izz="0.000011048923704800" />

Commit message: Fixed origin for wheel joint

File: balancingkit_description/robots/balancingkit.urdf.xacro (robot description, xacro)
@@ -13,10 +13,10 @@
   </xacro:base>
   <!-- Wheel -->
-  <xacro:wheel prefix="right" parent="base_link">
-    <origin xyz="0 0 0.0005" rpy="0 0 0"/>
+  <xacro:wheel prefix="right" parent="base_link" origin_x="-0.051">
+    <origin xyz="0.051 -0.02 -0.0097"/>
     <axis xyz="1 0 0"/>
   </xacro:wheel>
-  <xacro:wheel prefix="left" parent="base_link">
-    <origin xyz="0 0 0.0005" rpy="0 0 0"/>
+  <xacro:wheel prefix="left" parent="base_link" origin_x="0.051">
+    <origin xyz="-0.051 -0.02 -0.0097"/>
     <axis xyz="1 0 0"/>
   </xacro:wheel>

File: balancingkit_description/urdf/wheel/wheel.urdf.xacro (robot description, xacro)
@@ -6,5 +6,5 @@
   <property name="wheel_length" value="0.01"/> <!-- width? -->
   <property name="wheel_mass" value="0.0192200809141"/>
-  <xacro:macro name="wheel" params="prefix parent *joint_origin *joint_axis">
+  <xacro:macro name="wheel" params="prefix parent origin_x *joint_origin *joint_axis">
   <joint name="${prefix}_wheel_joint" type="continuous">
     <insert_block name="joint_origin"/>
@@ -18,4 +18,5 @@
   <link name="${prefix}_wheel">
     <visual>
+      <origin xyz="${origin_x} 0.02 0.0097" rpy="0 0 0"/>
       <geometry>
         <mesh filename="package://balancingkit_description/meshes/stl/wheel/balboa_balancing_robot_kit_wheel_${prefix}_m.stl"/>
@@ -24,9 +25,11 @@
     <collision>
       <!-- <insert_block name="joint_origin"/> -->
-        <geometry>
-          <mesh filename="package://balancingkit_description/meshes/stl/wheel/balboa_balancing_robot_kit_wheel_${prefix}_m.stl"/>
-        </geometry>
+      <origin xyz="${origin_x} 0.02 0.0097" rpy="0 0 0"/>
+      <geometry>
+        <mesh filename="package://balancingkit_description/meshes/stl/wheel/balboa_balancing_robot_kit_wheel_${prefix}_m.stl"/>
+      </geometry>
     </collision>
       <inertial>
+        <origin xyz="${origin_x} 0.02 0.0097" rpy="0 0 0"/>
         <mass value="${wheel_mass}"/>
         <inertia ixx="0.000021836231232000" ixy="0.000000000014016411" ixz="-0.000000000002704489" iyy="0.000011052671184900" iyz="-0.000000000002905832" izz="0.000011048923704800" />

Commit message: Add imu sensor and interface for it

File: balancingkit_description/robots/balancingkit.urdf.xacro (robot description, xacro)
@@ -6,4 +6,5 @@
   <xacro:include filename="$(find balancingkit_description)/urdf/body/body.urdf.xacro"/>
   <xacro:include filename="$(find balancingkit_description)/urdf/wheel/wheel.urdf.xacro"/>
+  <xacro:include filename="$(find balancingkit_description)/urdf/sensors/imu.urdf.xacro" />
   <!-- =============== Link & Joint =============== -->
   <!-- Base -->
@@ -21,4 +22,8 @@
     <axis xyz="1 0 0"/>
   </xacro:wheel>
+  <!-- Sensors -->
+  <xacro:imu_sensor prefix="imu" parent="base_link">
+    <origin xyz="0.02 0.048 0"/>
+  </xacro:imu_sensor>
   <!-- ===============  Transmission =============== -->
   <!-- PositionJointInterface: requires position -->
@@ -45,4 +50,5 @@
   <xacro:wheel_gazebo prefix="left"/>
   <!-- Sensors -->
+  <xacro:imu_gazebo prefix="imu"/>
   <balancingkit_on_gazebo/>
 </robot>

Commit message: Fixed wheel orgin

File: balancingkit_description/robots/balancingkit.urdf.xacro (robot description, xacro)
@@ -14,9 +14,9 @@
   </xacro:base>
   <!-- Wheel -->
-  <xacro:wheel prefix="right" parent="base_link" origin_x="-0.051">
+  <xacro:wheel prefix="right" parent="base_link" origin_x="-0.051" origin_x_2="0.051">
     <origin xyz="0.051 -0.02 -0.0097"/>
     <axis xyz="1 0 0"/>
   </xacro:wheel>
-  <xacro:wheel prefix="left" parent="base_link" origin_x="0.051">
+  <xacro:wheel prefix="left" parent="base_link" origin_x="0.051" origin_x_2="-0.051">
     <origin xyz="-0.051 -0.02 -0.0097"/>
     <axis xyz="1 0 0"/>

File: balancingkit_description/urdf/wheel/wheel.urdf.xacro (robot description, xacro)
@@ -6,6 +6,8 @@
   <property name="wheel_length" value="0.01"/> <!-- width? -->
   <property name="wheel_mass" value="0.0192200809141"/>
-  <xacro:macro name="wheel" params="prefix parent origin_x *joint_origin *joint_axis">
+  <xacro:macro name="wheel" params="prefix parent origin_x origin_x_2 *joint_origin *joint_axis">
   <joint name="${prefix}_wheel_joint" type="continuous">
+    <origin xyz="${origin_x} -0.02 -0.0097"/>
+    <axis xyz="1 0 0"/>
     <!-- <insert_block name="joint_origin"/> -->
     <insert_block name="joint_axis"/>
@@ -18,5 +20,5 @@
   <link name="${prefix}_wheel">
     <visual>
-      <origin xyz="${origin_x} 0.02 0.0097" rpy="0 0 0"/>
+      <origin xyz="${origin_x_2} 0.02 0.0097" rpy="0 0 0"/>
       <geometry>
         <mesh filename="package://balancingkit_description/meshes/stl/wheel/balboa_balancing_robot_kit_wheel_${prefix}_m.stl"/>
@@ -25,5 +27,5 @@
     <collision>
       <!-- <insert_block name="joint_origin"/> -->
-      <origin xyz="${origin_x} 0.02 0.0097" rpy="0 0 0"/>
+      <origin xyz="${origin_x_2} 0.02 0.0097" rpy="0 0 0"/>
       <geometry>
         <mesh filename="package://balancingkit_description/meshes/stl/wheel/balboa_balancing_robot_kit_wheel_${prefix}_m.stl"/>
@@ -31,5 +33,6 @@
     </collision>
       <inertial>
-        <origin xyz="${origin_x} 0.02 0.0097" rpy="0 0 0"/>
+        <origin xyz="${origin_x_2} 0.02 0.0097" rpy="0 0 0"/>
+        <origin xyz="0 0 0"/>
         <mass value="${wheel_mass}"/>
         <inertia ixx="0.000021836231232000" ixy="0.000000000014016411" ixz="-0.000000000002704489" iyy="0.000011052671184900" iyz="-0.000000000002905832" izz="0.000011048923704800" />

Commit message: Fixed some of bugs

File: balancingkit_description/robots/balancingkit.urdf.xacro (robot description, xacro)
@@ -11,5 +11,6 @@
   <link name="base_footprint"/>
   <xacro:base parent="base_footprint">
-    <origin xyz="0 0.02 0.0097"/>
+    <!--<origin xyz="0 0.02 0.0097"/>-->
+    <origin xyz="0 0 0"/>
   </xacro:base>
   <!-- Wheel -->
@@ -32,9 +33,9 @@
   <!-- VelocityJointInterface: requires position, velocity -->
   <!-- for DiffDriveController -->
-  <xacro:wheel_trans prefix="right" interface="hardware_interface/VelocityJointInterface"/>
-  <xacro:wheel_trans prefix="left" interface="hardware_interface/VelocityJointInterface"/>
+  <!-- <xacro:wheel_trans prefix="right" interface="hardware_interface/VelocityJointInterface"/> -->
+  <!-- <xacro:wheel_trans prefix="left" interface="hardware_interface/VelocityJointInterface"/> -->
   <!-- EffortJointInterface: requires position, velocity, effort -->
-  <!-- <xacro:wheel_trans prefix="right" interface="hardware_interface/EffortJointInterface"/> -->
-  <!-- <xacro:wheel_trans prefix="left" interface="hardware_interface/EffortJointInterface"/> -->
+  <xacro:wheel_trans prefix="right" interface="hardware_interface/EffortJointInterface"/>
+  <xacro:wheel_trans prefix="left" interface="hardware_interface/EffortJointInterface"/>
   <!-- =============== Gazebo =============== -->
   <gazebo>

File: balancingkit_description/urdf/wheel/wheel.urdf.xacro (robot description, xacro)
@@ -34,5 +34,4 @@
       <inertial>
         <origin xyz="${origin_x_2} 0.02 0.0097" rpy="0 0 0"/>
-        <origin xyz="0 0 0"/>
         <mass value="${wheel_mass}"/>
         <inertia ixx="0.000021836231232000" ixy="0.000000000014016411" ixz="-0.000000000002704489" iyy="0.000011052671184900" iyz="-0.000000000002905832" izz="0.000011048923704800" />
